File: ingenico/ingenico.kicad_pcb (KiCad board)
At the start: 2 copper layers, 56.2 x 93.9 mm, 0 parts

Commit message: Add files via upload
Other:
- board text added: "1"
- board text added: "10"
- board text added: "11"
- board text added: "12"
- board text added: "13"
- board text added: "14"
- board text added: "15"
- board text added: "16"
- board text added: "17"
- board text added: "18"
- board text added: "19"
- board text added: "2"
- board text added: "20"
- board text added: "21"
- board text added: "22"
- board text added: "23"
- board text added: "24"
- board text added: "25"
- board text added: "26"
- board text added: "27"
- board text added: "28"
- board text added: "29"
- board text added: "3"
- board text added: "30"
- board text added: "4"
- board text added: "5"
- board text added: "6"
- board text added: "7"
- board text added: "8"
- board text added: "9"
Changed lines of the file:
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@@
   (general
     (thickness 1.6)
-    (drawings 378)
+    (drawings 408)
     (tracks 0)
     (zones 0)
@@
     (uvia_drill 0.1)
   )
+  (gr_text 30 (at 129.722185 132.710086) (layer F.SilkS)
+    (effects (font (size 0.6 0.6) (thickness 0.08)))
+  )
+  (gr_text 29 (at 112.75 133.3) (layer F.SilkS)
+    (effects (font (size 0.6 0.6) (thickness 0.08)))
+  )
+  (gr_text 28 (at 95.8 132.7) (layer F.SilkS)
+    (effects (font (size 0.6 0.6) (thickness 0.08)))
+  )
+  (gr_text 27 (at 121.85 128.6) (layer F.SilkS)
+    (effects (font (size 0.6 0.6) (thickness 0.08)))
+  )
+  (gr_text 26 (at 103.75 128.6) (layer F.SilkS)
+    (effects (font (size 0.6 0.6) (thickness 0.08)))
+  )
+  (gr_text 25 (at 130.05 124.15) (layer F.SilkS)
+    (effects (font (size 0.6 0.6) (thickness 0.08)))
+  )
+  (gr_text 24 (at 112.747374 124.83504) (layer F.SilkS)
+    (effects (font (size 0.6 0.6) (thickness 0.08)))
+  )
+  (gr_text 23 (at 95.45 124.15) (layer F.SilkS)
+    (effects (font (size 0.6 0.6) (thickness 0.08)))
+  )
+  (gr_text 22 (at 122.05 120.55) (layer F.SilkS)
+    (effects (font (size 0.6 0.6) (thickness 0.08)))
+  )
+  (gr_text 21 (at 103.6 120.55) (layer F.SilkS)
+    (effects (font (size 0.6 0.6) (thickness 0.08)))
+  )
+  (gr_text 20 (at 130.3 116.1) (layer F.SilkS)
+    (effects (font (size 0.6 0.6) (thickness 0.08)))
+  )
+  (gr_text 19 (at 112.747374 116.74752) (layer F.SilkS)
+    (effects (font (size 0.6 0.6) (thickness 0.08)))
+  )
+  (gr_text 18 (at 95.181349 116.071056) (layer F.SilkS)
+    (effects (font (size 0.6 0.6) (thickness 0.08)))
+  )
+  (gr_text 17 (at 122.223433 112.522248) (layer F.SilkS)
+    (effects (font (size 0.6 0.6) (thickness 0.08)))
+  )
+  (gr_text 16 (at 103.4 112.5) (layer F.SilkS)
+    (effects (font (size 0.6 0.6) (thickness 0.08)))
+  )
+  (gr_text 15 (at 130.65 108) (layer F.SilkS)
+    (effects (font (size 0.6 0.6) (thickness 0.08)))
+  )
+  (gr_text 14 (at 112.75 108.75) (layer F.SilkS)
+    (effects (font (size 0.6 0.6) (thickness 0.08)))
+  )
+  (gr_text 13 (at 95 108) (layer F.SilkS)
+    (effects (font (size 0.6 0.6) (thickness 0.08)))
+  )
+  (gr_text 12 (at 130.65 99.9) (layer F.SilkS)
+    (effects (font (size 0.6 0.6) (thickness 0.08)))
+  )
+  (gr_text 11 (at 112.7 100.7) (layer F.SilkS)
+    (effects (font (size 0.6 0.6) (thickness 0.08)))
+  )
+  (gr_text 10 (at 94.8 99.85) (layer F.SilkS)
+    (effects (font (size 0.6 0.6) (thickness 0.08)))
+  )
+  (gr_text 9 (at 133.2 93.95) (layer F.SilkS)
+    (effects (font (size 0.6 0.6) (thickness 0.08)))
+  )
+  (gr_text 8 (at 112.65 93.7) (layer F.SilkS)
+    (effects (font (size 0.6 0.6) (thickness 0.08)))
+  )
+  (gr_text 7 (at 89.9 93.85) (layer F.SilkS)
+    (effects (font (size 0.6 0.6) (thickness 0.08)))
+  )
+  (gr_text 6 (at 132.372161 87.313459) (layer F.SilkS)
+    (effects (font (size 0.6 0.6) (thickness 0.08)))
+  )
+  (gr_text 5 (at 122.2 87.7) (layer F.SilkS)
+    (effects (font (size 0.6 0.6) (thickness 0.08)))
+  )
+  (gr_text 4 (at 112.7 87.7) (layer F.SilkS)
+    (effects (font (size 0.6 0.6) (thickness 0.08)))
+  )
+  (gr_text 3 (at 103.085806 87.692051) (layer F.SilkS)
+    (effects (font (size 0.6 0.6) (thickness 0.08)))
+  )
+  (gr_text 2 (at 92.90269 87.316017) (layer F.SilkS)
+    (effects (font (size 0.6 0.6) (thickness 0.08)))
+  )
+  (gr_text 1 (at 112.7 81.7) (layer F.SilkS)
+    (effects (font (size 0.6 0.6) (thickness 0.08)))
+  )
   (gr_line (start 113.955865 137.975586) (end 114.294661 137.975587) (layer Edge.Cuts) (width 0.2))
